Commit message: - up to s6_launch_file_instructions

File: ros2_ws2_vis_sim/src/practice_robot_description/urdf/_GlobalConfigs.urdf.xacro (robot description, xacro)
@@ -13,3 +13,31 @@
         <color rgba="0 0 0.5 1"/>
     </material>
+    <!-- wikipedia.org/wiki/List_of_moments_of_inertia#List_of_3D_inertia_tensors -->
+    <xacro:macro name="box_inertia" params="m x y z o_xyz o_rpy">
+        <inertial>
+            <mass value="${m}" />
+            <origin xyz="${o_xyz}" rpy="${o_rpy}" />
+            <inertia ixx="${(m/12) * (z*z + y*y)}" ixy="0" ixz="0"
+                     iyy="${(m/12) * (x*x + z*z)}" iyz="0"
+                     izz="${(m/12) * (x*x + y*y)}" />
+        </inertial>
+    </xacro:macro>
+    <xacro:macro name="cylinder_inertia" params="m r l o_xyz o_rpy">
+        <inertial>
+            <mass value="${m}" />
+            <origin xyz="${o_xyz}" rpy="${o_rpy}" />
+            <inertia ixx="${(m/12) * (3*r*r + l*l)}" ixy="0" ixz="0"
+                     iyy="${(m/12) * (3*r*r + l*l)}" iyz="0"
+                     izz="${(m/2) * (r*r)}" />
+        </inertial>
+    </xacro:macro>
+    <xacro:macro name="sphere_inertia" params="m r o_xyz o_rpy">
+        <inertial>
+            <mass value="${m}" />
+            <origin xyz="${o_xyz}" rpy="${o_rpy}" />
+            <inertia ixx="${(2/5) * m * r * r}" ixy="0" ixz="0"
+                     iyy="${(2/5) * m * r * r}" iyz="0"
+                     izz="${(2/5) * m * r * r}" />
+        </inertial>
+    </xacro:macro>
 </robot>

Commit message: - debugged the to give fixed link to the placeholder nodes that don't   need inertia

File: ros2_ws2_vis_sim/src/practice_robot_description/urdf/_GlobalConfigs.urdf.xacro (robot description, xacro)
@@ -29,5 +29,5 @@
             <inertia ixx="${(m/12) * (3*r*r + l*l)}" ixy="0" ixz="0"
                      iyy="${(m/12) * (3*r*r + l*l)}" iyz="0"
-                     izz="${(m/2) * (r*r)}" />
+                     izz="${(m/2)  * (r*r)}" />
         </inertial>
     </xacro:macro>
@@ -36,7 +36,7 @@
             <mass value="${m}" />
             <origin xyz="${o_xyz}" rpy="${o_rpy}" />
-            <inertia ixx="${(2/5) * m * r * r}" ixy="0" ixz="0"
-                     iyy="${(2/5) * m * r * r}" iyz="0"
-                     izz="${(2/5) * m * r * r}" />
+            <inertia ixx="${(2*m/5) * (r*r)}" ixy="0" ixz="0"
+                     iyy="${(2*m/5) * (r*r)}" iyz="0"
+                     izz="${(2*m/5) * (r*r)}" />
         </inertial>
     </xacro:macro>

File: ros2_ws2_vis_sim/src/practice_robot_description/urdf/practice.gazebo.urdf.xacro (robot description, xacro)
@@ -35,9 +35,8 @@
     </link>
     <link name="base_footprint"/>
-    <joint name="base_joint" type="continuous">
+    <joint name="base_joint" type="fixed">
         <parent link="base_footprint"/>
         <child link="base_link"/>
         <origin xyz="0 0 ${wheel_height}" rpy="0 0 0"/>
-        <axis xyz="0 0 1"/>
     </joint>
     <link name="right_wheel_link">

Commit message: - naming reorganization

File: ros2_ws2_vis_sim/src/practice_robot_description/urdf/_GlobalConfigs.urdf.xacro (robot description, xacro)
@@ -16,27 +16,27 @@
     <xacro:macro name="box_inertia" params="m x y z o_xyz o_rpy">
         <inertial>
-            <mass value="${m}" />
-            <origin xyz="${o_xyz}" rpy="${o_rpy}" />
+            <mass value="${m}"/>
+            <origin xyz="${o_xyz}" rpy="${o_rpy}"/>
             <inertia ixx="${(m/12) * (z*z + y*y)}" ixy="0" ixz="0"
                      iyy="${(m/12) * (x*x + z*z)}" iyz="0"
-                     izz="${(m/12) * (x*x + y*y)}" />
+                     izz="${(m/12) * (x*x + y*y)}"/>
         </inertial>
     </xacro:macro>
     <xacro:macro name="cylinder_inertia" params="m r l o_xyz o_rpy">
         <inertial>
-            <mass value="${m}" />
-            <origin xyz="${o_xyz}" rpy="${o_rpy}" />
+            <mass value="${m}"/>
+            <origin xyz="${o_xyz}" rpy="${o_rpy}"/>
             <inertia ixx="${(m/12) * (3*r*r + l*l)}" ixy="0" ixz="0"
                      iyy="${(m/12) * (3*r*r + l*l)}" iyz="0"
-                     izz="${(m/2)  * (r*r)}" />
+                     izz="${(m/2)  * (r*r)}"/>
         </inertial>
     </xacro:macro>
     <xacro:macro name="sphere_inertia" params="m r o_xyz o_rpy">
         <inertial>
-            <mass value="${m}" />
-            <origin xyz="${o_xyz}" rpy="${o_rpy}" />
+            <mass value="${m}"/>
+            <origin xyz="${o_xyz}" rpy="${o_rpy}"/>
             <inertia ixx="${(2*m/5) * (r*r)}" ixy="0" ixz="0"
                      iyy="${(2*m/5) * (r*r)}" iyz="0"
-                     izz="${(2*m/5) * (r*r)}" />
+                     izz="${(2*m/5) * (r*r)}"/>
         </inertial>
     </xacro:macro>

File: ros2_ws2_vis_sim/src/practice_robot_description/urdf/diffCart.gazebo.urdf.xacro (robot description, xacro)
@@ -1,5 +1,5 @@
 <?xml version="1.0"?>
 <!-- ======================================================================================================== -->
-<robot name="practice" xmlns:xacro="http://www.ros.org/wiki/xacro">
+<robot name="diffCart" xmlns:xacro="http://www.ros.org/wiki/xacro">
     <xacro:include filename="_GlobalConfigs.urdf.xacro"/>
     <xacro:property name="base_x" value="0.6"/>

File: ros2_ws2_vis_sim/src/practice_robot_description/urdf/diffCart.urdf.xacro (robot description, xacro)
@@ -1,4 +1,4 @@
 <?xml version="1.0"?>
-<robot name="practice" xmlns:xacro="http://www.ros.org/wiki/xacro">
+<robot name="diffCart" xmlns:xacro="http://www.ros.org/wiki/xacro">
     <xacro:include filename="_GlobalConfigs.urdf.xacro"/>
     <xacro:property name="base_x" value="0.6"/>

Commit message: - initial file for diffCartWithArm

File: ros2_ws2_vis_sim/src/practice_robot_description/urdf/_GlobalConfigs.urdf.xacro (robot description, xacro)
@@ -12,4 +12,10 @@
     <material name="blue">
         <color rgba="0 0 0.5 1"/>
+    </material>
+    <material name="orange">
+        <color rgba="1 0.647 0 1"/>
+    </material>
+    <material name="yellow">
+        <color rgba="1 1 0 1"/>
     </material>
     <!-- wikipedia.org/wiki/List_of_moments_of_inertia#List_of_3D_inertia_tensors -->
