Commit message: - rvis test of arduinobot.urdf.xacro

File: ros2_ws4_manipulators/src/robot_description/urdf/arduinobot.urdf.xacro (robot description, xacro)
@@ -1,7 +1,6 @@
 <?xml version="1.0"?>
+<!-- reference from  Antonio Brandi, "Robotics and ROS 2 - Learn by Doing! Manipulators" (Udemy) -->
 <robot xmlns:xacro="http://www.ros.org/wiki/xacro" name="arduinobot">
-    <!-- Useful XACRO Variables (Properties) -->
-    <xacro:property name="PI" value="3.14159265359" />
-    <xacro:property name="effort" value="30.0" />
+    <xacro:property name="effort"   value="30.0" />
     <xacro:property name="velocity" value="10.0" />
     <!-- Links -->
@@ -11,5 +10,5 @@
             <origin rpy="0 0 0" xyz="-0.5 -0.5 0"/>
             <geometry>
-                <mesh filename="package://arduinobot_description/meshes/basement.STL" scale="0.01 0.01 0.01"/>
+                <mesh filename="package://robot_description/mesh/basement.STL" scale="0.01 0.01 0.01"/>
             </geometry>
         </visual>
@@ -19,5 +18,5 @@
             <origin rpy="0 0 0" xyz="-0.39 -0.39 -0.56"/>
             <geometry>
-                <mesh filename="package://arduinobot_description/meshes/base_plate.STL" scale="0.01 0.01 0.01"/>
+                <mesh filename="package://robot_description/mesh/base_plate.STL" scale="0.01 0.01 0.01"/>
             </geometry>
         </visual>
@@ -25,7 +24,7 @@
     <link name="forward_drive_arm">
         <visual>
-            <origin rpy=" 0 -${PI / 2} ${PI / 2}" xyz="0.19 0.06 -0.08"/>
+            <origin rpy=" 0 -${pi/2} ${pi/2}" xyz="0.19 0.06 -0.08"/>
             <geometry>
-                <mesh filename="package://arduinobot_description/meshes/forward_drive_arm.STL" scale="0.01 0.01 0.01"/>
+                <mesh filename="package://robot_description/mesh/forward_drive_arm.STL" scale="0.01 0.01 0.01"/>
             </geometry>
         </visual>
@@ -33,7 +32,7 @@
     <link name="horizontal_arm">
         <visual>
-            <origin rpy="${PI / 2} 0 ${PI / 2}" xyz="-0.03 -0.4 -0.06"/>
+            <origin rpy="${pi/2} 0 ${pi/2}" xyz="-0.03 -0.4 -0.06"/>
             <geometry>
-                <mesh filename="package://arduinobot_description/meshes/horizontal_arm.STL" scale="0.01 0.01 0.01"/>
+                <mesh filename="package://robot_description/mesh/horizontal_arm.STL" scale="0.01 0.01 0.01"/>
             </geometry>
         </visual>
@@ -41,7 +40,7 @@
     <link name="claw_support">
         <visual>
-            <origin rpy="0 0 ${PI / 2}" xyz="0 -0.05 -0.15"/>
+            <origin rpy="0 0 ${pi/2}" xyz="0 -0.05 -0.15"/>
             <geometry>
-                <mesh filename="package://arduinobot_description/meshes/claw_support.STL" scale="0.01 0.01 0.01"/>
+                <mesh filename="package://robot_description/mesh/claw_support.STL" scale="0.01 0.01 0.01"/>
             </geometry>
         </visual>
@@ -49,7 +48,7 @@
     <link name="gripper_right">
         <visual>
-            <origin rpy="0 0 -${PI / 2}" xyz="-0.1 0.50 -0.1"/>
+            <origin rpy="0 0 -${pi/2}" xyz="-0.1 0.50 -0.1"/>
             <geometry>
-                <mesh filename="package://arduinobot_description/meshes/right_finger.STL" scale="0.01 0.01 0.01"/>
+                <mesh filename="package://robot_description/mesh/right_finger.STL" scale="0.01 0.01 0.01"/>
             </geometry>
         </visual>
@@ -57,7 +56,7 @@
     <link name="gripper_left">
         <visual>
-            <origin rpy="0 0 -${PI / 2}" xyz="-0.04 0.50 -0.1"/>
+            <origin rpy="0 0 -${pi/2}" xyz="-0.04 0.50 -0.1"/>
             <geometry>
-                <mesh filename="package://arduinobot_description/meshes/left_finger.STL" scale="0.01 0.01 0.01"/>
+                <mesh filename="package://robot_description/mesh/left_finger.STL" scale="0.01 0.01 0.01"/>
             </geometry>
         </visual>
@@ -67,5 +66,5 @@
             <origin rpy="-1.57 0 -1.57" xyz="-0.1 0.125 0.15"/>
             <geometry>
-                <mesh filename="package://arduinobot_description/meshes/pi_camera.STL" scale="0.01 0.01 0.01"/>
+                <mesh filename="package://robot_description/mesh/pi_camera.STL" scale="0.01 0.01 0.01"/>
             </geometry>
         </visual>
@@ -82,5 +81,5 @@
         <origin xyz="0 0 0.307"/>
         <axis xyz="0 0 1"/>
-        <limit lower="-${PI / 2}" upper="${PI / 2}"
+        <limit lower="-${pi/2}" upper="${pi/2}"
                effort="${effort}" velocity="${velocity}"/>
     </joint>
@@ -90,5 +89,5 @@
         <origin xyz="-0.02 0 0.35"/>
         <axis xyz="1 0 0"/>
-        <limit lower="-${PI / 2}" upper="${PI / 2}"
+        <limit lower="-${pi/2}" upper="${pi/2}"
                 effort="${effort}" velocity="${velocity}"/>
     </joint>
@@ -98,5 +97,5 @@
         <origin xyz="0 0 0.8"/>
         <axis xyz="1 0 0"/>
-        <limit lower="-${PI / 2}" upper="${PI / 2}"
+        <limit lower="-${pi/2}" upper="${pi/2}"
                effort="${effort}" velocity="${velocity}"/>
     </joint>
@@ -111,5 +110,5 @@
         <origin xyz="-0.04 0.13 -0.1"/>
         <axis xyz="0 0 1"/>
-        <limit lower="-${PI / 2}" upper="0.0"
+        <limit lower="-${pi/2}" upper="0.0"
                effort="${effort}" velocity="${velocity}"/>
     </joint>
@@ -119,5 +118,5 @@
         <origin xyz="-0.22 0.13 -0.1"/>
         <axis xyz="0 0 1"/>
-        <limit lower="0.0" upper="${PI / 2}"
+        <limit lower="0.0" upper="${pi/2}"
                effort="${effort}" velocity="${velocity}"/>
         <mimic joint="joint_4" multiplier="-1"/>
