Commit message: - enabling the gazebo for the course project

File: ros2_ws4_manipulators/src/robot_description/urdf/_GlobalConfigs.urdf.xacro (robot description, xacro)
@@ -47,11 +47,3 @@
         </inertial>
     </xacro:macro>
-    <xacro:macro name="lazy_inertia" params="m">
-        <inertial>
-            <mass value="${m}"/>
-            <inertia ixx="${m/12}" ixy="0" ixz="0"
-                     iyy="${m/12}" iyz="0"
-                     izz="${m/12}"/>
-        </inertial>
-    </xacro:macro>
 </robot>

Commit message: - add color - add physics engine option - debug

File: ros2_ws4_manipulators/src/robot_description/urdf/_GlobalConfigs.urdf.xacro (robot description, xacro)
@@ -47,3 +47,11 @@
         </inertial>
     </xacro:macro>
+    <xacro:macro name="lazy_inertia" params="m">
+        <inertial>
+            <mass value="${m}"/>
+            <inertia ixx="${m/12}" ixy="0" ixz="0"
+                     iyy="${m/12}" iyz="0"
+                     izz="${m/12}"/>
+        </inertial>
+    </xacro:macro>
 </robot>

File: ros2_ws4_manipulators/src/robot_description/urdf/arduinobot.gazebo.urdf.xacro (robot description, xacro)
@@ -15,4 +15,5 @@
                 <mesh filename="package://robot_description/mesh/basement.STL" scale="0.01 0.01 0.01"/>
             </geometry>
+            <material name="red"/>
         </visual>
         <collision>
@@ -30,4 +31,5 @@
                 <mesh filename="package://robot_description/mesh/base_plate.STL" scale="0.01 0.01 0.01"/>
             </geometry>
+            <material name="blue"/>
         </visual>
         <collision>
@@ -45,4 +47,5 @@
                 <mesh filename="package://robot_description/mesh/forward_drive_arm.STL" scale="0.01 0.01 0.01"/>
             </geometry>
+            <material name="green"/>
         </visual>
         <collision>
@@ -60,4 +63,5 @@
                 <mesh filename="package://robot_description/mesh/horizontal_arm.STL" scale="0.01 0.01 0.01"/>
             </geometry>
+            <material name="green"/>
         </visual>
         <collision>
@@ -75,4 +79,5 @@
                 <mesh filename="package://robot_description/mesh/claw_support.STL" scale="0.01 0.01 0.01"/>
             </geometry>
+            <material name="blue"/>
         </visual>
         <collision>
@@ -90,4 +95,5 @@
                 <mesh filename="package://robot_description/mesh/right_finger.STL" scale="0.01 0.01 0.01"/>
             </geometry>
+            <material name="red"/>
         </visual>
         <collision>
@@ -105,4 +111,5 @@
                 <mesh filename="package://robot_description/mesh/left_finger.STL" scale="0.01 0.01 0.01"/>
             </geometry>
+            <material name="red"/>
         </visual>
         <collision>
@@ -120,4 +127,5 @@
                 <mesh filename="package://robot_description/mesh/pi_camera.STL" scale="0.01 0.01 0.01"/>
             </geometry>
+            <material name="green"/>
         </visual>
         <collision>
@@ -138,5 +146,5 @@
     <joint name ="joint_1" type="revolute">
         <parent link="base_link"/>
-        <child link = "base_plate"/>
+        <child link="base_plate"/>
         <origin xyz="0 0 0.307"/>
         <axis xyz="0 0 1"/>
@@ -146,5 +154,5 @@
     <joint name ="joint_2" type="revolute">
         <parent link="base_plate"/>
-        <child link = "forward_drive_arm"/>
+        <child link="forward_drive_arm"/>
         <origin xyz="-0.02 0 0.35"/>
         <axis xyz="1 0 0"/>
@@ -154,5 +162,5 @@
     <joint name ="joint_3" type="revolute">
         <parent link="forward_drive_arm"/>
-        <child link = "horizontal_arm"/>
+        <child link="horizontal_arm"/>
         <origin xyz="0 0 0.8"/>
         <axis xyz="1 0 0"/>
@@ -162,10 +170,10 @@
     <joint name ="horizontal_arm_to_claw_support" type="fixed">
         <parent link="horizontal_arm"/>
-        <child link = "claw_support"/>
+        <child link="claw_support"/>
         <origin xyz="0 0.82 0"/>
     </joint>
     <joint name ="joint_4" type="revolute">
         <parent link="claw_support"/>
-        <child link = "gripper_right"/>
+        <child link="gripper_right"/>
         <origin xyz="-0.04 0.13 -0.1"/>
         <axis xyz="0 0 1"/>
@@ -175,5 +183,5 @@
     <joint name ="joint_5" type="revolute">
         <parent link="claw_support"/>
-        <child link = "gripper_left"/>
+        <child link="gripper_left"/>
         <origin xyz="-0.22 0.13 -0.1"/>
         <axis xyz="0 0 1"/>
@@ -184,40 +192,9 @@
     <joint name ="rgb_camera_joint" type="fixed">
         <parent link="base_link"/>
-        <child link = "rgb_camera"/>
+        <child link="rgb_camera"/>
         <origin xyz="0 0.45 0.2" rpy="0 -0.5 1.57"/>
     </joint>
 <!-- ======================================================================================================== -->
     <!-- Gazebo -->
-    <gazebo reference="rgb_camera">
-        <sensor name="camera" type="camera">
-            <pose>0 0 0 0 0 0</pose>
-            <visualize>true</visualize>
-            <always_on>1</always_on>
-            <update_rate>10</update_rate>
-            <topic>camera/image</topic>
-            <camera>
-                <horizontal_fov>1.3962634</horizontal_fov>
-                <image>
-                    <width>640</width>
-                    <height>480</height>
-                    <format>R8G8B8</format>
-                </image>
-                <clip>
-                    <near>0.1</near>
-                    <far>15</far>
-                </clip>
-                <noise>
-                    <type>gaussian</type>
-                    <mean>0.0</mean>
-                    <stddev>0.007</stddev>
-                </noise>
-                <optical_frame_id>camera_link_optical</optical_frame_id>
-                <camera_info_topic>camera/camera_info</camera_info_topic>
-            </camera>
-        </sensor>
-        <plugin name="libgazebo_ros_camera.so" filename="gazebo_ros::Camera">
-            <frame_name>rgb_camera</frame_name>
-        </plugin>
-    </gazebo>
 <!-- ======================================================================================================== -->
 </robot>
