Commit message: - updating to use ros2_controller for the course

File: ros2_ws4_manipulators/src/robot_description/urdf/arduinobot.rvis.urdf.xacro (robot description, xacro)
@@ -1,10 +1,7 @@
 <?xml version="1.0"?>
-<!-- ======================================================================================================== -->
 <!-- reference from  Antonio Brandi, "Robotics and ROS 2 - Learn by Doing! Manipulators" (Udemy) -->
 <robot xmlns:xacro="http://www.ros.org/wiki/xacro" name="arduinobot">
-    <xacro:include filename="_GlobalConfigs.urdf.xacro"/>
     <xacro:property name="effort"   value="30.0" />
     <xacro:property name="velocity" value="10.0" />
-<!-- ======================================================================================================== -->
     <!-- Links -->
     <link name="world"/>
@@ -15,13 +12,5 @@
                 <mesh filename="package://robot_description/mesh/basement.STL" scale="0.01 0.01 0.01"/>
             </geometry>
-            <material name="red"/>
         </visual>
-        <collision>
-            <origin rpy="0 0 0" xyz="-0.5 -0.5 0"/>
-            <geometry>
-                <mesh filename="package://robot_description/mesh/basement.STL" scale="0.01 0.01 0.01"/>
-            </geometry>
-        </collision>
-        <xacro:lazy_inertia m="1.0"/>
     </link>
     <link name="base_plate">
@@ -31,13 +20,5 @@
                 <mesh filename="package://robot_description/mesh/base_plate.STL" scale="0.01 0.01 0.01"/>
             </geometry>
-            <material name="blue"/>
         </visual>
-        <collision>
-            <origin rpy="0 0 0" xyz="-0.39 -0.39 -0.56"/>
-            <geometry>
-                <mesh filename="package://robot_description/mesh/base_plate.STL" scale="0.01 0.01 0.01"/>
-            </geometry>
-        </collision>
-        <xacro:lazy_inertia m="0.1"/>
     </link>
     <link name="forward_drive_arm">
@@ -47,13 +28,5 @@
                 <mesh filename="package://robot_description/mesh/forward_drive_arm.STL" scale="0.01 0.01 0.01"/>
             </geometry>
-            <material name="green"/>
         </visual>
-        <collision>
-            <origin rpy=" 0 -${pi/2} ${pi/2}" xyz="0.19 0.06 -0.08"/>
-            <geometry>
-                <mesh filename="package://robot_description/mesh/forward_drive_arm.STL" scale="0.01 0.01 0.01"/>
-            </geometry>
-        </collision>
-        <xacro:lazy_inertia m="0.1"/>
     </link>
     <link name="horizontal_arm">
@@ -63,13 +36,5 @@
                 <mesh filename="package://robot_description/mesh/horizontal_arm.STL" scale="0.01 0.01 0.01"/>
             </geometry>
-            <material name="green"/>
         </visual>
-        <collision>
-            <origin rpy="${pi/2} 0 ${pi/2}" xyz="-0.03 -0.4 -0.06"/>
-            <geometry>
-                <mesh filename="package://robot_description/mesh/horizontal_arm.STL" scale="0.01 0.01 0.01"/>
-            </geometry>
-        </collision>
-        <xacro:lazy_inertia m="0.1"/>
     </link>
     <link name="claw_support">
@@ -79,13 +44,5 @@
                 <mesh filename="package://robot_description/mesh/claw_support.STL" scale="0.01 0.01 0.01"/>
             </geometry>
-            <material name="blue"/>
         </visual>
-        <collision>
-            <origin rpy="0 0 ${pi/2}" xyz="0 -0.05 -0.15"/>
-            <geometry>
-                <mesh filename="package://robot_description/mesh/claw_support.STL" scale="0.01 0.01 0.01"/>
-            </geometry>
-        </collision>
-        <xacro:lazy_inertia m="0.05"/>
     </link>
     <link name="gripper_right">
@@ -95,13 +52,5 @@
                 <mesh filename="package://robot_description/mesh/right_finger.STL" scale="0.01 0.01 0.01"/>
             </geometry>
-            <material name="red"/>
         </visual>
-        <collision>
-            <origin rpy="0 0 -${pi/2}" xyz="-0.1 0.50 -0.1"/>
-            <geometry>
-                <mesh filename="package://robot_description/mesh/right_finger.STL" scale="0.01 0.01 0.01"/>
-            </geometry>
-        </collision>
-        <xacro:lazy_inertia m="0.01"/>
     </link>
     <link name="gripper_left">
@@ -111,13 +60,5 @@
                 <mesh filename="package://robot_description/mesh/left_finger.STL" scale="0.01 0.01 0.01"/>
             </geometry>
-            <material name="red"/>
         </visual>
-        <collision>
-            <origin rpy="0 0 -${pi/2}" xyz="-0.04 0.50 -0.1"/>
-            <geometry>
-                <mesh filename="package://robot_description/mesh/left_finger.STL" scale="0.01 0.01 0.01"/>
-            </geometry>
-        </collision>
-        <xacro:lazy_inertia m="0.01"/>
     </link>
     <link name="rgb_camera">
@@ -127,15 +68,6 @@
                 <mesh filename="package://robot_description/mesh/pi_camera.STL" scale="0.01 0.01 0.01"/>
             </geometry>
-            <material name="green"/>
         </visual>
-        <collision>
-            <origin rpy="-1.57 0 -1.57" xyz="-0.1 0.125 0.15"/>
-            <geometry>
-                <mesh filename="package://robot_description/mesh/pi_camera.STL" scale="0.01 0.01 0.01"/>
-            </geometry>
-        </collision>
-        <xacro:lazy_inertia m="0.1"/>
     </link>
-<!-- ======================================================================================================== -->
     <!-- Joints -->
     <joint name="virtual_joint" type="fixed">
@@ -146,5 +78,5 @@
     <joint name ="joint_1" type="revolute">
         <parent link="base_link"/>
-        <child link="base_plate"/>
+        <child link = "base_plate"/>
         <origin xyz="0 0 0.307"/>
         <axis xyz="0 0 1"/>
@@ -154,5 +86,5 @@
     <joint name ="joint_2" type="revolute">
         <parent link="base_plate"/>
-        <child link="forward_drive_arm"/>
+        <child link = "forward_drive_arm"/>
         <origin xyz="-0.02 0 0.35"/>
         <axis xyz="1 0 0"/>
@@ -162,5 +94,5 @@
     <joint name ="joint_3" type="revolute">
         <parent link="forward_drive_arm"/>
-        <child link="horizontal_arm"/>
+        <child link = "horizontal_arm"/>
         <origin xyz="0 0 0.8"/>
         <axis xyz="1 0 0"/>
@@ -170,10 +102,10 @@
     <joint name ="horizontal_arm_to_claw_support" type="fixed">
         <parent link="horizontal_arm"/>
-        <child link="claw_support"/>
+        <child link = "claw_support"/>
         <origin xyz="0 0.82 0"/>
     </joint>
     <joint name ="joint_4" type="revolute">
         <parent link="claw_support"/>
-        <child link="gripper_right"/>
+        <child link = "gripper_right"/>
         <origin xyz="-0.04 0.13 -0.1"/>
         <axis xyz="0 0 1"/>
@@ -183,5 +115,5 @@
     <joint name ="joint_5" type="revolute">
         <parent link="claw_support"/>
-        <child link="gripper_left"/>
+        <child link = "gripper_left"/>
         <origin xyz="-0.22 0.13 -0.1"/>
         <axis xyz="0 0 1"/>
@@ -192,9 +124,6 @@
     <joint name ="rgb_camera_joint" type="fixed">
         <parent link="base_link"/>
-        <child link="rgb_camera"/>
+        <child link = "rgb_camera"/>
         <origin xyz="0 0.45 0.2" rpy="0 -0.5 1.57"/>
     </joint>
-<!-- ======================================================================================================== -->
-    <!-- Gazebo -->
-<!-- ======================================================================================================== -->
 </robot>

File: ros2_ws4_manipulators/src/robot_description/urdf/arduinobot.urdf.xacro (robot description, xacro)
@@ -1,7 +1,12 @@
 <?xml version="1.0"?>
+<!-- ======================================================================================================== -->
 <!-- reference from  Antonio Brandi, "Robotics and ROS 2 - Learn by Doing! Manipulators" (Udemy) -->
 <robot xmlns:xacro="http://www.ros.org/wiki/xacro" name="arduinobot">
+    <xacro:include filename="$(find robot_description)/urdf/_GlobalConfigs.urdf.xacro"/>
+    <xacro:include filename="$(find robot_description)/urdf/arduinobot.gazebo.xacro"/>
+    <xacro:include filename="$(find robot_description)/urdf/arduinobot.ros2_control.xacro"/>
     <xacro:property name="effort"   value="30.0" />
     <xacro:property name="velocity" value="10.0" />
+<!-- ======================================================================================================== -->
     <!-- Links -->
     <link name="world"/>
@@ -12,5 +17,13 @@
                 <mesh filename="package://robot_description/mesh/basement.STL" scale="0.01 0.01 0.01"/>
             </geometry>
-        </visual>
+            <material name="red"/>
+        </visual>
+        <collision>
+            <origin rpy="0 0 0" xyz="-0.5 -0.5 0"/>
+            <geometry>
+                <mesh filename="package://robot_description/mesh/basement.STL" scale="0.01 0.01 0.01"/>
+            </geometry>
+        </collision>
+        <xacro:lazy_inertia m="1.0"/>
     </link>
     <link name="base_plate">
@@ -20,5 +33,13 @@
                 <mesh filename="package://robot_description/mesh/base_plate.STL" scale="0.01 0.01 0.01"/>
             </geometry>
-        </visual>
+            <material name="blue"/>
+        </visual>
+        <collision>
+            <origin rpy="0 0 0" xyz="-0.39 -0.39 -0.56"/>
+            <geometry>
+                <mesh filename="package://robot_description/mesh/base_plate.STL" scale="0.01 0.01 0.01"/>
+            </geometry>
+        </collision>
+        <xacro:lazy_inertia m="0.1"/>
     </link>
     <link name="forward_drive_arm">
@@ -28,5 +49,13 @@
                 <mesh filename="package://robot_description/mesh/forward_drive_arm.STL" scale="0.01 0.01 0.01"/>
             </geometry>
-        </visual>
+            <material name="green"/>
+        </visual>
+        <collision>
+            <origin rpy=" 0 -${pi/2} ${pi/2}" xyz="0.19 0.06 -0.08"/>
+            <geometry>
+                <mesh filename="package://robot_description/mesh/forward_drive_arm.STL" scale="0.01 0.01 0.01"/>
+            </geometry>
+        </collision>
+        <xacro:lazy_inertia m="0.1"/>
     </link>
     <link name="horizontal_arm">
@@ -36,5 +65,13 @@
                 <mesh filename="package://robot_description/mesh/horizontal_arm.STL" scale="0.01 0.01 0.01"/>
             </geometry>
-        </visual>
+            <material name="green"/>
+        </visual>
+        <collision>
+            <origin rpy="${pi/2} 0 ${pi/2}" xyz="-0.03 -0.4 -0.06"/>
+            <geometry>
+                <mesh filename="package://robot_description/mesh/horizontal_arm.STL" scale="0.01 0.01 0.01"/>
+            </geometry>
+        </collision>
+        <xacro:lazy_inertia m="0.1"/>
     </link>
     <link name="claw_support">
@@ -44,5 +81,13 @@
                 <mesh filename="package://robot_description/mesh/claw_support.STL" scale="0.01 0.01 0.01"/>
             </geometry>
-        </visual>
+            <material name="blue"/>
+        </visual>
+        <collision>
+            <origin rpy="0 0 ${pi/2}" xyz="0 -0.05 -0.15"/>
+            <geometry>
+                <mesh filename="package://robot_description/mesh/claw_support.STL" scale="0.01 0.01 0.01"/>
+            </geometry>
+        </collision>
+        <xacro:lazy_inertia m="0.05"/>
     </link>
     <link name="gripper_right">
@@ -52,5 +97,13 @@
                 <mesh filename="package://robot_description/mesh/right_finger.STL" scale="0.01 0.01 0.01"/>
             </geometry>
-        </visual>
+            <material name="red"/>
+        </visual>
+        <collision>
+            <origin rpy="0 0 -${pi/2}" xyz="-0.1 0.50 -0.1"/>
+            <geometry>
+                <mesh filename="package://robot_description/mesh/right_finger.STL" scale="0.01 0.01 0.01"/>
+            </geometry>
+        </collision>
+        <xacro:lazy_inertia m="0.01"/>
     </link>
     <link name="gripper_left">
@@ -60,5 +113,13 @@
                 <mesh filename="package://robot_description/mesh/left_finger.STL" scale="0.01 0.01 0.01"/>
             </geometry>
-        </visual>
+            <material name="red"/>
+        </visual>
+        <collision>
+            <origin rpy="0 0 -${pi/2}" xyz="-0.04 0.50 -0.1"/>
+            <geometry>
+                <mesh filename="package://robot_description/mesh/left_finger.STL" scale="0.01 0.01 0.01"/>
+            </geometry>
+        </collision>
+        <xacro:lazy_inertia m="0.01"/>
     </link>
     <link name="rgb_camera">
@@ -68,6 +129,15 @@
                 <mesh filename="package://robot_description/mesh/pi_camera.STL" scale="0.01 0.01 0.01"/>
             </geometry>
-        </visual>
-    </link>
+            <material name="green"/>
+        </visual>
+        <collision>
+            <origin rpy="-1.57 0 -1.57" xyz="-0.1 0.125 0.15"/>
+            <geometry>
+                <mesh filename="package://robot_description/mesh/pi_camera.STL" scale="0.01 0.01 0.01"/>
+            </geometry>
+        </collision>
+        <xacro:lazy_inertia m="0.1"/>
+    </link>
+<!-- ======================================================================================================== -->
     <!-- Joints -->
     <joint name="virtual_joint" type="fixed">
@@ -78,5 +148,5 @@
     <joint name ="joint_1" type="revolute">
         <parent link="base_link"/>
-        <child link = "base_plate"/>
+        <child link="base_plate"/>
         <origin xyz="0 0 0.307"/>
         <axis xyz="0 0 1"/>
@@ -86,5 +156,5 @@
     <joint name ="joint_2" type="revolute">
         <parent link="base_plate"/>
-        <child link = "forward_drive_arm"/>
+        <child link="forward_drive_arm"/>
         <origin xyz="-0.02 0 0.35"/>
         <axis xyz="1 0 0"/>
@@ -94,5 +164,5 @@
     <joint name ="joint_3" type="revolute">
         <parent link="forward_drive_arm"/>
-        <child link = "horizontal_arm"/>
+        <child link="horizontal_arm"/>
         <origin xyz="0 0 0.8"/>
         <axis xyz="1 0 0"/>
@@ -102,10 +172,10 @@
     <joint name ="horizontal_arm_to_claw_support" type="fixed">
         <parent link="horizontal_arm"/>
-        <child link = "claw_support"/>
+        <child link="claw_support"/>
         <origin xyz="0 0.82 0"/>
     </joint>
     <joint name ="joint_4" type="revolute">
         <parent link="claw_support"/>
-        <child link = "gripper_right"/>
+        <child link="gripper_right"/>
         <origin xyz="-0.04 0.13 -0.1"/>
         <axis xyz="0 0 1"/>
@@ -115,5 +185,5 @@
     <joint name ="joint_5" type="revolute">
         <parent link="claw_support"/>
-        <child link = "gripper_left"/>
+        <child link="gripper_left"/>
         <origin xyz="-0.22 0.13 -0.1"/>
         <axis xyz="0 0 1"/>
@@ -124,6 +194,7 @@
     <joint name ="rgb_camera_joint" type="fixed">
         <parent link="base_link"/>
-        <child link = "rgb_camera"/>
+        <child link="rgb_camera"/>
         <origin xyz="0 0.45 0.2" rpy="0 -0.5 1.57"/>
     </joint>
+<!-- ======================================================================================================== -->
 </robot>
