Commit message: - robot_build instead of robot_description

File: ros2_ws4_manipulators/src/robot_build/urdf/arduinobot.rvis.urdf.xacro (robot description, xacro)
@@ -10,5 +10,5 @@
             <origin rpy="0 0 0" xyz="-0.5 -0.5 0"/>
             <geometry>
-                <mesh filename="package://robot_description/mesh/basement.STL" scale="0.01 0.01 0.01"/>
+                <mesh filename="package://robot_build/mesh/basement.STL" scale="0.01 0.01 0.01"/>
             </geometry>
         </visual>
@@ -18,5 +18,5 @@
             <origin rpy="0 0 0" xyz="-0.39 -0.39 -0.56"/>
             <geometry>
-                <mesh filename="package://robot_description/mesh/base_plate.STL" scale="0.01 0.01 0.01"/>
+                <mesh filename="package://robot_build/mesh/base_plate.STL" scale="0.01 0.01 0.01"/>
             </geometry>
         </visual>
@@ -26,5 +26,5 @@
             <origin rpy=" 0 -${pi/2} ${pi/2}" xyz="0.19 0.06 -0.08"/>
             <geometry>
-                <mesh filename="package://robot_description/mesh/forward_drive_arm.STL" scale="0.01 0.01 0.01"/>
+                <mesh filename="package://robot_build/mesh/forward_drive_arm.STL" scale="0.01 0.01 0.01"/>
             </geometry>
         </visual>
@@ -34,5 +34,5 @@
             <origin rpy="${pi/2} 0 ${pi/2}" xyz="-0.03 -0.4 -0.06"/>
             <geometry>
-                <mesh filename="package://robot_description/mesh/horizontal_arm.STL" scale="0.01 0.01 0.01"/>
+                <mesh filename="package://robot_build/mesh/horizontal_arm.STL" scale="0.01 0.01 0.01"/>
             </geometry>
         </visual>
@@ -42,5 +42,5 @@
             <origin rpy="0 0 ${pi/2}" xyz="0 -0.05 -0.15"/>
             <geometry>
-                <mesh filename="package://robot_description/mesh/claw_support.STL" scale="0.01 0.01 0.01"/>
+                <mesh filename="package://robot_build/mesh/claw_support.STL" scale="0.01 0.01 0.01"/>
             </geometry>
         </visual>
@@ -50,5 +50,5 @@
             <origin rpy="0 0 -${pi/2}" xyz="-0.1 0.50 -0.1"/>
             <geometry>
-                <mesh filename="package://robot_description/mesh/right_finger.STL" scale="0.01 0.01 0.01"/>
+                <mesh filename="package://robot_build/mesh/right_finger.STL" scale="0.01 0.01 0.01"/>
             </geometry>
         </visual>
@@ -58,5 +58,5 @@
             <origin rpy="0 0 -${pi/2}" xyz="-0.04 0.50 -0.1"/>
             <geometry>
-                <mesh filename="package://robot_description/mesh/left_finger.STL" scale="0.01 0.01 0.01"/>
+                <mesh filename="package://robot_build/mesh/left_finger.STL" scale="0.01 0.01 0.01"/>
             </geometry>
         </visual>
@@ -66,5 +66,5 @@
             <origin rpy="-1.57 0 -1.57" xyz="-0.1 0.125 0.15"/>
             <geometry>
-                <mesh filename="package://robot_description/mesh/pi_camera.STL" scale="0.01 0.01 0.01"/>
+                <mesh filename="package://robot_build/mesh/pi_camera.STL" scale="0.01 0.01 0.01"/>
             </geometry>
         </visual>

File: ros2_ws4_manipulators/src/robot_build/urdf/arduinobot.urdf.xacro (robot description, xacro)
@@ -3,7 +3,7 @@
 <!-- reference from  Antonio Brandi, "Robotics and ROS 2 - Learn by Doing! Manipulators" (Udemy) -->
 <robot xmlns:xacro="http://www.ros.org/wiki/xacro" name="arduinobot">
-    <xacro:include filename="$(find robot_description)/urdf/_GlobalConfigs.urdf.xacro"/>
-    <xacro:include filename="$(find robot_description)/urdf/arduinobot.gazebo.xacro"/>
-    <xacro:include filename="$(find robot_description)/urdf/arduinobot.ros2_control.xacro"/>
+    <xacro:include filename="$(find robot_build)/urdf/_GlobalConfigs.urdf.xacro"/>
+    <xacro:include filename="$(find robot_build)/urdf/arduinobot.gazebo.xacro"/>
+    <xacro:include filename="$(find robot_build)/urdf/arduinobot.ros2_control.xacro"/>
     <xacro:property name="effort"   value="30.0" />
     <xacro:property name="velocity" value="10.0" />
@@ -15,5 +15,5 @@
             <origin rpy="0 0 0" xyz="-0.5 -0.5 0"/>
             <geometry>
-                <mesh filename="package://robot_description/mesh/basement.STL" scale="0.01 0.01 0.01"/>
+                <mesh filename="package://robot_build/mesh/basement.STL" scale="0.01 0.01 0.01"/>
             </geometry>
             <material name="red"/>
@@ -22,5 +22,5 @@
             <origin rpy="0 0 0" xyz="-0.5 -0.5 0"/>
             <geometry>
-                <mesh filename="package://robot_description/mesh/basement.STL" scale="0.01 0.01 0.01"/>
+                <mesh filename="package://robot_build/mesh/basement.STL" scale="0.01 0.01 0.01"/>
             </geometry>
         </collision>
@@ -31,5 +31,5 @@
             <origin rpy="0 0 0" xyz="-0.39 -0.39 -0.56"/>
             <geometry>
-                <mesh filename="package://robot_description/mesh/base_plate.STL" scale="0.01 0.01 0.01"/>
+                <mesh filename="package://robot_build/mesh/base_plate.STL" scale="0.01 0.01 0.01"/>
             </geometry>
             <material name="blue"/>
@@ -38,5 +38,5 @@
             <origin rpy="0 0 0" xyz="-0.39 -0.39 -0.56"/>
             <geometry>
-                <mesh filename="package://robot_description/mesh/base_plate.STL" scale="0.01 0.01 0.01"/>
+                <mesh filename="package://robot_build/mesh/base_plate.STL" scale="0.01 0.01 0.01"/>
             </geometry>
         </collision>
@@ -47,5 +47,5 @@
             <origin rpy=" 0 -${pi/2} ${pi/2}" xyz="0.19 0.06 -0.08"/>
             <geometry>
-                <mesh filename="package://robot_description/mesh/forward_drive_arm.STL" scale="0.01 0.01 0.01"/>
+                <mesh filename="package://robot_build/mesh/forward_drive_arm.STL" scale="0.01 0.01 0.01"/>
             </geometry>
             <material name="green"/>
@@ -54,5 +54,5 @@
             <origin rpy=" 0 -${pi/2} ${pi/2}" xyz="0.19 0.06 -0.08"/>
             <geometry>
-                <mesh filename="package://robot_description/mesh/forward_drive_arm.STL" scale="0.01 0.01 0.01"/>
+                <mesh filename="package://robot_build/mesh/forward_drive_arm.STL" scale="0.01 0.01 0.01"/>
             </geometry>
         </collision>
@@ -63,5 +63,5 @@
             <origin rpy="${pi/2} 0 ${pi/2}" xyz="-0.03 -0.4 -0.06"/>
             <geometry>
-                <mesh filename="package://robot_description/mesh/horizontal_arm.STL" scale="0.01 0.01 0.01"/>
+                <mesh filename="package://robot_build/mesh/horizontal_arm.STL" scale="0.01 0.01 0.01"/>
             </geometry>
             <material name="green"/>
@@ -70,5 +70,5 @@
             <origin rpy="${pi/2} 0 ${pi/2}" xyz="-0.03 -0.4 -0.06"/>
             <geometry>
-                <mesh filename="package://robot_description/mesh/horizontal_arm.STL" scale="0.01 0.01 0.01"/>
+                <mesh filename="package://robot_build/mesh/horizontal_arm.STL" scale="0.01 0.01 0.01"/>
             </geometry>
         </collision>
@@ -79,5 +79,5 @@
             <origin rpy="0 0 ${pi/2}" xyz="0 -0.05 -0.15"/>
             <geometry>
-                <mesh filename="package://robot_description/mesh/claw_support.STL" scale="0.01 0.01 0.01"/>
+                <mesh filename="package://robot_build/mesh/claw_support.STL" scale="0.01 0.01 0.01"/>
             </geometry>
             <material name="blue"/>
@@ -86,5 +86,5 @@
             <origin rpy="0 0 ${pi/2}" xyz="0 -0.05 -0.15"/>
             <geometry>
-                <mesh filename="package://robot_description/mesh/claw_support.STL" scale="0.01 0.01 0.01"/>
+                <mesh filename="package://robot_build/mesh/claw_support.STL" scale="0.01 0.01 0.01"/>
             </geometry>
         </collision>
@@ -95,5 +95,5 @@
             <origin rpy="0 0 -${pi/2}" xyz="-0.1 0.50 -0.1"/>
             <geometry>
-                <mesh filename="package://robot_description/mesh/right_finger.STL" scale="0.01 0.01 0.01"/>
+                <mesh filename="package://robot_build/mesh/right_finger.STL" scale="0.01 0.01 0.01"/>
             </geometry>
             <material name="red"/>
@@ -102,5 +102,5 @@
             <origin rpy="0 0 -${pi/2}" xyz="-0.1 0.50 -0.1"/>
             <geometry>
-                <mesh filename="package://robot_description/mesh/right_finger.STL" scale="0.01 0.01 0.01"/>
+                <mesh filename="package://robot_build/mesh/right_finger.STL" scale="0.01 0.01 0.01"/>
             </geometry>
         </collision>
@@ -111,5 +111,5 @@
             <origin rpy="0 0 -${pi/2}" xyz="-0.04 0.50 -0.1"/>
             <geometry>
-                <mesh filename="package://robot_description/mesh/left_finger.STL" scale="0.01 0.01 0.01"/>
+                <mesh filename="package://robot_build/mesh/left_finger.STL" scale="0.01 0.01 0.01"/>
             </geometry>
             <material name="red"/>
@@ -118,5 +118,5 @@
             <origin rpy="0 0 -${pi/2}" xyz="-0.04 0.50 -0.1"/>
             <geometry>
-                <mesh filename="package://robot_description/mesh/left_finger.STL" scale="0.01 0.01 0.01"/>
+                <mesh filename="package://robot_build/mesh/left_finger.STL" scale="0.01 0.01 0.01"/>
             </geometry>
         </collision>
@@ -127,5 +127,5 @@
             <origin rpy="-1.57 0 -1.57" xyz="-0.1 0.125 0.15"/>
             <geometry>
-                <mesh filename="package://robot_description/mesh/pi_camera.STL" scale="0.01 0.01 0.01"/>
+                <mesh filename="package://robot_build/mesh/pi_camera.STL" scale="0.01 0.01 0.01"/>
             </geometry>
             <material name="green"/>
@@ -134,5 +134,5 @@
             <origin rpy="-1.57 0 -1.57" xyz="-0.1 0.125 0.15"/>
             <geometry>
-                <mesh filename="package://robot_description/mesh/pi_camera.STL" scale="0.01 0.01 0.01"/>
+                <mesh filename="package://robot_build/mesh/pi_camera.STL" scale="0.01 0.01 0.01"/>
             </geometry>
         </collision>

File: ros2_ws4_manipulators/src/robot_build/urdf/arduinobot_test.urdf.xacro (robot description, xacro)
@@ -9,5 +9,5 @@
             <origin rpy="0 0 0" xyz="-0.5 -0.5 0"/>
             <geometry>
-                <mesh filename="package://robot_description/mesh/basement.STL" scale="0.01 0.01 0.01"/>
+                <mesh filename="package://robot_build/mesh/basement.STL" scale="0.01 0.01 0.01"/>
             </geometry>
         </visual>
@@ -17,5 +17,5 @@
             <origin rpy="0 0 0" xyz="-0.39 -0.39 -0.56"/>
             <geometry>
-                <mesh filename="package://robot_description/mesh/base_plate.STL" scale="0.01 0.01 0.01"/>
+                <mesh filename="package://robot_build/mesh/base_plate.STL" scale="0.01 0.01 0.01"/>
             </geometry>
         </visual>
