Commit message: - starting by adding in the urdf needed according to udemy Ch5

File: ros2_ws4_controller/src/my_robot_description/urdf/common_properties.xacro (robot description, xacro)
@@ -7,3 +7,9 @@
         <color rgba="0.5 0.5 0.5 1" />
     </material>
+    <material name="orange">
+        <color rgba="1.0 0.5 0 1" />
+    </material>
+    <material name="yellow">
+        <color rgba="1.0 1.0 0 1" />
+    </material>
 </robot>
