Commit message: - adjusted, now ready to put inertia type in urdf for gazebo sim

File: ros2_ws4_controller/src/my_robot_description/urdf/arm.ros2_control.xacro (robot description, xacro)
@@ -6,8 +6,8 @@
             <param name="calculate_dynamics">true</param-->
             <plugin>ma_robot_arm/HardwareInterfacePCA9685_arm</plugin>
-                <param name="joint1_servo_channel">2</param>
-                <param name="joint2_servo_channel">3</param>
-                <param name="pwm_min_microSec">600</param>
-                <param name="pwm_max_microSec">2400</param>
+            <param name="joint1_servo_channel">2</param>
+            <param name="joint2_servo_channel">3</param>
+            <param name="pwm_min_microSec">600</param>
+            <param name="pwm_max_microSec">2400</param>
         </hardware>
         <joint name="arm_joint1">

File: ros2_ws5_manipulator/src/my_robot_description/urdf/arduinobot.urdf.xacro (robot description, xacro)
@@ -3,5 +3,5 @@
 <!-- reference from  Antonio Brandi, "Robotics and ROS 2 - Learn by Doing! Manipulators" (Udemy) -->
 <robot xmlns:xacro="http://www.ros.org/wiki/xacro" name="arduinobot">
-    <xacro:include filename="$(find my_robot_description)/urdf/arduinobot_common_properties.urdf.xacro"/>
+    <xacro:include filename="$(find my_robot_description)/urdf/common_properties.xacro"/>
     <!-- xacro:include filename="$(find robot_build)/urdf/arduinobot.ros2_control.xacro"/-->
     <xacro:property name="effort"   value="30.0" />

File: ros2_ws5_manipulator/src/my_robot_description/urdf/common_properties.xacro (robot description, xacro)
@@ -18,4 +18,10 @@
     <material name="yellow">
         <color rgba="1 1 0 1"/>
+    </material>
+    <material name="dark_green">
+        <color rgba="0 0.4 0 1" />
+    </material>
+    <material name="light_green">
+        <color rgba="0 0.6 0 1" />
     </material>
     <!-- wikipedia.org/wiki/List_of_moments_of_inertia#List_of_3D_inertia_tensors -->

File: ros2_ws5_manipulator/src/my_robot_description/urdf/ma_robot.gazebo.xacro (robot description, xacro)
@@ -1,5 +1,5 @@
 <?xml version="1.0"?>
 <robot name="ma_robot" xmlns:xacro="http://www.ros.org/wiki/xacro">
-    <xacro:include filename="my_robot_common_properties.xacro" />
+    <xacro:include filename="common_properties.xacro" />
     <xacro:include filename="my_robot_arm.xacro" />
     <xacro:include filename="my_robot_gripper.xacro" />
@@ -9,4 +9,51 @@
         <origin xyz="0 0 0" rpy="0 0 0" />
     </joint>
+    <ros2_control name="GazeboInterface" type="system">
+        <hardware>
+            <plugin>gz_ros2_control/GazeboSimSystem</plugin>
+        </hardware>
+        <joint name="gripper_left_finger_joint">
+            <command_interface name="position"/>
+            <state_interface name="position">
+                <param name="initial_value">0.0</param>
+            </state_interface>
+        </joint>
+        <joint name="joint1">
+            <command_interface name="position"/>
+            <state_interface name="position">
+                <param name="initial_value">0.0</param>
+            </state_interface>
+        </joint>
+        <joint name="joint2">
+            <command_interface name="position"/>
+            <state_interface name="position">
+                <param name="initial_value">0.0</param>
+            </state_interface>
+        </joint>
+        <joint name="joint3">
+            <command_interface name="position"/>
+            <state_interface name="position">
+                <param name="initial_value">0.0</param>
+            </state_interface>
+        </joint>
+        <joint name="joint4">
+            <command_interface name="position"/>
+            <state_interface name="position">
+                <param name="initial_value">0.0</param>
+            </state_interface>
+        </joint>
+        <joint name="joint5">
+            <command_interface name="position"/>
+            <state_interface name="position">
+                <param name="initial_value">0.0</param>
+            </state_interface>
+        </joint>
+        <joint name="joint6">
+            <command_interface name="position"/>
+            <state_interface name="position">
+                <param name="initial_value">0.0</param>
+            </state_interface>
+        </joint>
+    </ros2_control>
     <gazebo>
         <plugin filename="gz_ros2_control-system" name="gz_ros2_control::GazeboSimROS2ControlPlugin">

File: ros2_ws5_manipulator/src/my_robot_description/urdf/ma_robot.urdf.xacro (robot description, xacro)
@@ -1,5 +1,5 @@
 <?xml version="1.0"?>
 <robot name="ma_robot" xmlns:xacro="http://www.ros.org/wiki/xacro">
-    <xacro:include filename="my_robot_common_properties.xacro" />
+    <xacro:include filename="common_properties.xacro" />
     <xacro:include filename="my_robot_arm.xacro" />
     <xacro:include filename="my_robot_gripper.xacro" />

File: ros2_ws5_manipulator/src/my_robot_description/urdf/my_robot.urdf.xacro (robot description, xacro)
@@ -1,5 +1,5 @@
 <?xml version="1.0"?>
 <robot name="my_robot" xmlns:xacro="http://www.ros.org/wiki/xacro">
-    <xacro:include filename="my_robot_common_properties.xacro" />
+    <xacro:include filename="common_properties.xacro" />
     <xacro:include filename="my_robot_arm.xacro" />
 </robot>
