Commit message: - adding moveit config for the arm+gripper

File: ros2_ws5_manipulator/src/my_robot_description/urdf/common_properties.xacro (robot description, xacro)
@@ -7,3 +7,9 @@
         <color rgba="0 0 0.5 1" />
     </material>
-</robot>
+    <material name="dark_green">
+        <color rgba="0 0.4 0 1" />
+    </material>
+    <material name="light_green">
+        <color rgba="0 0.6 0 1" />
+    </material>
+</robot>%
