Commit message: - added inertia, but joint don't seems to sync, cannot issue moveit command

File: ros2_ws5_manipulator/src/my_robot_description/urdf/my_robot_arm.xacro (robot description, xacro)
@@ -15,4 +15,6 @@
             <origin xyz="0 0 0.05" rpy="0 0 0" />
         </collision>
+        <xacro:box_inertia m="5.0" x="0.4" y="0.4" z="0.1"
+                           o_xyz="0 0 0.05" o_rpy="0 0 0" />
     </link>
     <link name="shoulder_link">
@@ -30,4 +32,6 @@
             <origin xyz="0 0 0.25" rpy="0 0 0" />
         </collision>
+        <xacro:box_inertia m="0.1" x="0.2" y="0.2" z="0.5"
+                           o_xyz="0 0 0.25" o_rpy="0 0 0" />
     </link>
     <link name="arm_link">
@@ -45,4 +49,6 @@
             <origin xyz="0 0 0.3" rpy="0 0 0" />
         </collision>
+        <xacro:box_inertia m="0.5" x="0.1" y="0.1" z="0.6"
+                           o_xyz="0 0 0.3" o_rpy="0 0 0" />
     </link>
     <link name="elbow_link">
@@ -60,4 +66,6 @@
             <origin xyz="0 0 0.05" rpy="0 0 0" />
         </collision>
+        <xacro:box_inertia m="0.1" x="0.1" y="0.1" z="0.1"
+                           o_xyz="0 0 0.05" o_rpy="0 0 0" />
     </link>
     <link name="forearm_link">
@@ -75,4 +83,6 @@
             <origin xyz="0 0 0.25" rpy="0 0 0" />
         </collision>
+        <xacro:box_inertia m="0.5" x="0.1" y="0.1" z="0.5"
+                           o_xyz="0 0 0.025" o_rpy="0 0 0" />
     </link>
     <link name="wrist_link">
@@ -90,4 +100,6 @@
             <origin xyz="0 0 0.025" rpy="0 0 0" />
         </collision>
+        <xacro:box_inertia m="0.1" x="0.1" y="0.1" z="0.5"
+                           o_xyz="0 0 0.025" o_rpy="0 0 0" />
     </link>
     <link name="hand_link">
@@ -105,4 +117,6 @@
             <origin xyz="0 0 0.01" rpy="0 0 0" />
         </collision>
+        <xacro:box_inertia m="0.1" x="0.1" y="0.1" z="0.2"
+                           o_xyz="0 0 0.01" o_rpy="0 0 0" />
     </link>
     <link name="tool_link" />
@@ -113,4 +127,5 @@
         <axis xyz="0 0 1" />
         <limit effort="1000.0" velocity="1.0" lower="-3.14" upper="3.14" />
+        <dynamics friction="0.05" damping="0.1" />
     </joint>
     <joint name="joint2" type="revolute">
@@ -120,4 +135,5 @@
         <axis xyz="0 1 0" />
         <limit effort="1000.0" velocity="1.0" lower="0" upper="2.5" />
+        <dynamics friction="0.05" damping="0.1" />
     </joint>
     <joint name="joint3" type="revolute">
@@ -127,4 +143,5 @@
         <axis xyz="0 1 0" />
         <limit effort="1000.0" velocity="1.0" lower="0" upper="2.5" />
+        <dynamics friction="0.05" damping="0.1" />
     </joint>
     <joint name="joint4" type="revolute">
@@ -134,4 +151,5 @@
         <axis xyz="0 0 1" />
         <limit effort="1000.0" velocity="1.0" lower="-3.14" upper="3.14" />
+        <dynamics friction="0.05" damping="0.1" />
     </joint>
     <joint name="joint5" type="revolute">
@@ -141,4 +159,5 @@
         <axis xyz="0 1 0" />
         <limit effort="1000.0" velocity="1.0" lower="-1.57" upper="1.57" />
+        <dynamics friction="0.05" damping="0.1" />
     </joint>
     <joint name="joint6" type="continuous">
@@ -147,4 +166,6 @@
         <origin xyz="0 0 0.05" rpy="0 0 0" />
         <axis xyz="0 0 1" />
+        <limit effort="1000.0" velocity="1.0" lower="-3.14" upper="3.14" />
+        <dynamics friction="0.05" damping="0.1" />
     </joint>
     <joint name="hand_tool_joint" type="fixed">

File: ros2_ws5_manipulator/src/my_robot_description/urdf/my_robot_gripper.xacro (robot description, xacro)
@@ -15,4 +15,6 @@
             <origin xyz="0 0 0.01" rpy="0 0 0" />
         </collision>
+        <xacro:box_inertia m="0.1" x="0.2" y="0.06" z="0.02"
+                           o_xyz="0 0 0.01" o_rpy="0 0 0" />
     </link>
     <link name="gripper_left_finger_link">
@@ -30,4 +32,6 @@
             <origin xyz="0 0 0.04" rpy="0 0 0" />
         </collision>
+        <xacro:box_inertia m="0.05" x="0.02" y="0.06" z="0.08"
+                           o_xyz="0 0 0.04" o_rpy="0 0 0" />
     </link>
     <link name="gripper_right_finger_link">
@@ -45,4 +49,6 @@
             <origin xyz="0 0 0.04" rpy="0 0 0" />
         </collision>
+        <xacro:box_inertia m="0.05" x="0.02" y="0.06" z="0.08"
+                           o_xyz="0 0 0.04" o_rpy="0 0 0" />
     </link>
     <joint name="gripper_left_finger_joint" type="prismatic">
